File: DC.kicad_sch (KiCad schematic)
At the start: 102 parts, among them J1 348302001, J2 348302001, J3 757570141, J4 PPTC021LFBN-RC, Q1 BSS806NE, Q2 BSS806NE, Q3 BSS806NE, Q4 BSS806NE, Q5 BSS806NE, U1 MCP2551-I-P, U2 100DP6T1B1M1QEH, U5 NUCLEO-F302R8, U6 C1F 250

Commit message: hello
Parts:
- S1, S2, S3: value LP6OA2ASRG -> LP11EE1NCSYG; footprint DriverControlsLib:LP6OA2ASRG -> DriverControlsLib:LP11EE1NCSYG; symbol DriverControlsLib:LP6OA2ASRG -> DriverControlsLib:LP11EE1NCSYG; Height 20.7 -> 23.25; Manufacturer_Part_Number LP6OA2ASRG -> LP11EE1NCSYG; Mouser Part Number 612-LP6OA2ASRG -> 612-LP11EE1NCSYG; Mouser Price/Stock https://www.mouser.co.uk/ProductDetail/E-Switch/LP6OA2ASRG?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 -> https://www.mouser.co.uk/ProductDetail/E-Switch/LP11EE1NCSY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
Connections:
- net GND: no longer S1.MH1, S1.MH2, S1.MH3, S1.MH4, S2.MH1, S2.MH2, S2.MH3, S2.MH4, S3.MH1, S3.MH2, S3.MH3, S3.MH4
- no-connect marks 53 -> 47
